Commit message: [EDIT] Reference and simulation

File: urdf/stair.urdf (robot description, URDF)
Before this commit: robot stair_skeleton, 2 links, 1 joints
Links:
- link stair_link: geometry collision box size=1.0 2.0 0.1; visual box size=1.0 2.0 0.1

Commit message: (fix) trajectories, midpoint, covariance

File: urdf/stair.urdf (robot description, URDF)
Before this commit: robot stair_2_steps, 5 links, 4 joints
Joints:
- joint fixed_to_world: origin xyz=0.45 0 0 rpy=0 0 0 -> xyz=0.60 0 0 rpy=0 0 0
